File: dmxhat.kicad_pcb (KiCad board)
At the start: 2 copper layers, 73.7 x 53.3 mm, 24 parts, among them J1 XLR5, J2 Conn_01x03, P1 Power, P2 Analog, P3 Digital, P4 Digital, P5 CONN_01X01, P6 CONN_01X01, P7 CONN_01X01, SW1 SW_DIP_x05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

Commit message: Update to revision 1.1
Parts:
- removed REF**: OSHW-Logo_5.7x6mm_SilkScreen, Symbol:OSHW-Logo_5.7x6mm_SilkScreen
- added G***: LOGO, Logo:license, F.Cu at (156.1, 111.1)
- added J3: XLR3, Connector_Audio:Jack_XLR_Neutrik_NC3FAH1-DA_Horizontal, F.Cu at (119.0, 107.3)
- moved J1 3.83 mm to (123.4, 107.3)
Routing:
- net /DMX+: track 79.3 -> 67.5 mm
- net GND: track 139.5 -> 131.9 mm
- net /DMX-: track 81.3 -> 85.0 mm
Other:
- outline, holes or cut-outs redrawn
- board text added: "JLCJLCJLCJLC"
